File: pcb/pcb.kicad_pcb (KiCad board)
At the start: 2 copper layers, 489.6 x 170.7 mm, 286 parts, among them J1 Conn_01x08_Socket, J2 Conn_01x02_Female, U1 YAAJ_WeAct_BlackPill_Part_Lik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

Commit message: attempting to add RGB
Parts:
- removed 10U1: 10U, MX_Only:MXOnly-10U-Hotswap-ReversedStabilizers
- removed BZ1: Buzzer, Buzzer_Beeper:Buzzer_TDK_PS1240P02BT_D12.2mm_H6.5mm
- removed D18: BAV70, Keebio-Parts:SOT-23_Handsoldering
- removed MX047: MX-NoLED, MX_Only:MXOnly-2.25U-Hotswap
- removed MX051.125: MX-NoLED, MX_Only:MXOnly-1.25U-Hotswap
- removed MX062: MX-NoLED, MX_Only:MXOnly-2.75U-Hotswap
- removed MX063: MX-NoLED, MX_Only:MXOnly-2U-Hotswap
- removed MX066.100, MX077, MX087, MX089.100, MX099, MX109.100, MX121, MX136, MX137: MX-NoLED, MX_Only:MXOnly-1U-Hotswap
- removed MX117: MX-NoLED, MX_Only:MXOnly-1.5U-Hotswap
- removed MX132.225: MX-NoLED, MX_Only:MXOnly-2.25U-Hotswap-ReversedStabilizers
- removed R1, R2: 470, Keebio-Parts:Resistor-Hybrid-Back
- removed R3: R_22K, Keebio-Parts:Resistor-Hybrid
- added C1: 100n, schizobovine:C_0603_1608Metric, B.Cu at (305.5, 36.2)
- added FID1: Fiducial, schizobovine:COW, F.Cu at (173.7, 174.9)
- added LD1: WS2812B, schizobovine:LED_SK6812MINI_PLCC4_3.1x2.7mm_P1.75mm_reverse_mount, F.Cu at (285.8, 35.7)
- added LD10: WS2812B, schizobovine:LED_SK6812MINI_PLCC4_3.1x2.7mm_P1.75mm_reverse_mount, F.Cu at (114.3, 35.7)
- added LD100: WS2812B, schizobovine:LED_SK6812MINI_PLCC4_3.1x2.7mm_P1.75mm_reverse_mount, F.Cu at (214.3, 159.1)
- added LD101: WS2812B, schizobovine:LED_SK6812MINI_PLCC4_3.1x2.7mm_P1.75mm_reverse_mount, F.Cu at (233.4, 159.1)
- added LD102: WS2812B, schizobovine:LED_SK6812MINI_PLCC4_3.1x2.7mm_P1.75mm_reverse_mount, F.Cu at (252.4, 159.1)
- added LD103: WS2812B, schizobovine:LED_SK6812MINI_PLCC4_3.1x2.7mm_P1.75mm_reverse_mount, F.Cu at (271.5, 159.1)
- added LD104: WS2812B, schizobovine:LED_SK6812MINI_PLCC4_3.1x2.7mm_P1.75mm_reverse_mount, F.Cu at (290.5, 149.3)
- added LD105: WS2812B, schizobovine:LED_SK6812MINI_PLCC4_3.1x2.7mm_P1.75mm_reverse_mount, F.Cu at (307.2, 159.1)
- added LD106: WS2812B, schizobovine:LED_SK6812MINI_PLCC4_3.1x2.7mm_P1.75mm_reverse_mount, F.Cu at (351.8, 159.1)
- added LD107: WS2812B, schizobovine:LED_SK6812MINI_PLCC4_3.1x2.7mm_P1.75mm_reverse_mount, F.Cu at (370.8, 159.1)
- added LD108: WS2812B, schizobovine:LED_SK6812MINI_PLCC4_3.1x2.7mm_P1.75mm_reverse_mount, F.Cu at (389.9, 159.1)
- added LD109: WS2812B, schizobovine:LED_SK6812MINI_PLCC4_3.1x2.7mm_P1.75mm_reverse_mount, F.Cu at (417.8, 159.1)
- added LD11: WS2812B, schizobovine:LED_SK6812MINI_PLCC4_3.1x2.7mm_P1.75mm_reverse_mount, F.Cu at (95.2, 35.7)
- added LD110: WS2812B, schizobovine:LED_SK6812MINI_PLCC4_3.1x2.7mm_P1.75mm_reverse_mount, F.Cu at (436.9, 159.1)
- added LD111: WS2812B, schizobovine:LED_SK6812MINI_PLCC4_3.1x2.7mm_P1.75mm_reverse_mount, F.Cu at (455.9, 159.1)
- added LD112: WS2812B, schizobovine:LED_SK6812MINI_PLCC4_3.1x2.7mm_P1.75mm_reverse_mount, F.Cu at (475.0, 169.4)
- added LD113: WS2812B, schizobovine:LED_SK6812MINI_PLCC4_3.1x2.7mm_P1.75mm_reverse_mount, F.Cu at (455.9, 179.7)
- added LD114: WS2812B, schizobovine:LED_SK6812MINI_PLCC4_3.1x2.7mm_P1.75mm_reverse_mount, F.Cu at (427.3, 179.7)
- added LD115: WS2812B, schizobovine:LED_SK6812MINI_PLCC4_3.1x2.7mm_P1.75mm_reverse_mount, F.Cu at (370.8, 179.7)
- added LD116: WS2812B, schizobovine:LED_SK6812MINI_PLCC4_3.1x2.7mm_P1.75mm_reverse_mount, F.Cu at (319.1, 179.7)
- added LD117: WS2812B, schizobovine:LED_SK6812MINI_PLCC4_3.1x2.7mm_P1.75mm_reverse_mount, F.Cu at (271.5, 179.7)
- added LD118: WS2812B, schizobovine:LED_SK6812MINI_PLCC4_3.1x2.7mm_P1.75mm_reverse_mount, F.Cu at (190.5, 179.7)
- added LD119: WS2812B, schizobovine:LED_SK6812MINI_PLCC4_3.1x2.7mm_P1.75mm_reverse_mount, F.Cu at (109.5, 179.7)
- added LD12: WS2812B, schizobovine:LED_SK6812MINI_PLCC4_3.1x2.7mm_P1.75mm_reverse_mount, F.Cu at (76.2, 35.7)
- added LD120: WS2812B, schizobovine:LED_SK6812MINI_PLCC4_3.1x2.7mm_P1.75mm_reverse_mount, F.Cu at (61.9, 179.7)
- added LD121: WS2812B, schizobovine:LED_SK6812MINI_PLCC4_3.1x2.7mm_P1.75mm_reverse_mount, F.Cu at (29.2, 179.7)
- added LD122: WS2812B, schizobovine:LED_SK6812MINI_PLCC4_3.1x2.7mm_P1.75mm_reverse_mount, F.Cu at (10.2, 179.7)
- added LD13: WS2812B, schizobovine:LED_SK6812MINI_PLCC4_3.1x2.7mm_P1.75mm_reverse_mount, F.Cu at (76.2, 56.3)
- added LD14: WS2812B, schizobovine:LED_SK6812MINI_PLCC4_3.1x2.7mm_P1.75mm_reverse_mount, F.Cu at (95.2, 56.3)
- added LD15: WS2812B, schizobovine:LED_SK6812MINI_PLCC4_3.1x2.7mm_P1.75mm_reverse_mount, F.Cu at (114.3, 56.3)
- added LD16: WS2812B, schizobovine:LED_SK6812MINI_PLCC4_3.1x2.7mm_P1.75mm_reverse_mount, F.Cu at (133.3, 56.3)
- added LD17: WS2812B, schizobovine:LED_SK6812MINI_PLCC4_3.1x2.7mm_P1.75mm_reverse_mount, F.Cu at (152.4, 56.3)
- added LD18: WS2812B, schizobovine:LED_SK6812MINI_PLCC4_3.1x2.7mm_P1.75mm_reverse_mount, F.Cu at (171.4, 56.3)
- added LD19: WS2812B, schizobovine:LED_SK6812MINI_PLCC4_3.1x2.7mm_P1.75mm_reverse_mount, F.Cu at (190.5, 56.3)
- added LD2: WS2812B, schizobovine:LED_SK6812MINI_PLCC4_3.1x2.7mm_P1.75mm_reverse_mount, F.Cu at (266.7, 35.7)
- added LD20: WS2812B, schizobovine:LED_SK6812MINI_PLCC4_3.1x2.7mm_P1.75mm_reverse_mount, F.Cu at (209.6, 56.3)
- added LD21: WS2812B, schizobovine:LED_SK6812MINI_PLCC4_3.1x2.7mm_P1.75mm_reverse_mount, F.Cu at (228.6, 56.3)
- added LD22: WS2812B, schizobovine:LED_SK6812MINI_PLCC4_3.1x2.7mm_P1.75mm_reverse_mount, F.Cu at (247.7, 56.3)
- added LD23: WS2812B, schizobovine:LED_SK6812MINI_PLCC4_3.1x2.7mm_P1.75mm_reverse_mount, F.Cu at (266.7, 56.3)
- added LD24: WS2812B, schizobovine:LED_SK6812MINI_PLCC4_3.1x2.7mm_P1.75mm_reverse_mount, F.Cu at (285.8, 56.3)
- added LD25: WS2812B, schizobovine:LED_SK6812MINI_PLCC4_3.1x2.7mm_P1.75mm_reverse_mount, F.Cu at (475.0, 97.4)
- added LD26: WS2812B, schizobovine:LED_SK6812MINI_PLCC4_3.1x2.7mm_P1.75mm_reverse_mount, F.Cu at (455.9, 97.4)
- added LD27: WS2812B, schizobovine:LED_SK6812MINI_PLCC4_3.1x2.7mm_P1.75mm_reverse_mount, F.Cu at (436.9, 97.4)
- added LD28: WS2812B, schizobovine:LED_SK6812MINI_PLCC4_3.1x2.7mm_P1.75mm_reverse_mount, F.Cu at (417.8, 97.4)
- added LD29: WS2812B, schizobovine:LED_SK6812MINI_PLCC4_3.1x2.7mm_P1.75mm_reverse_mount, F.Cu at (389.9, 97.4)
- added LD3: WS2812B, schizobovine:LED_SK6812MINI_PLCC4_3.1x2.7mm_P1.75mm_reverse_mount, F.Cu at (247.7, 35.7)
- added LD30: WS2812B, schizobovine:LED_SK6812MINI_PLCC4_3.1x2.7mm_P1.75mm_reverse_mount, F.Cu at (370.8, 97.4)
- added LD31: WS2812B, schizobovine:LED_SK6812MINI_PLCC4_3.1x2.7mm_P1.75mm_reverse_mount, F.Cu at (351.8, 97.4)
- added LD32: WS2812B, schizobovine:LED_SK6812MINI_PLCC4_3.1x2.7mm_P1.75mm_reverse_mount, F.Cu at (314.3, 97.4)
- added LD33: WS2812B, schizobovine:LED_SK6812MINI_PLCC4_3.1x2.7mm_P1.75mm_reverse_mount, F.Cu at (285.8, 97.4)
- added LD34: WS2812B, schizobovine:LED_SK6812MINI_PLCC4_3.1x2.7mm_P1.75mm_reverse_mount, F.Cu at (266.7, 97.4)
- added LD35: WS2812B, schizobovine:LED_SK6812MINI_PLCC4_3.1x2.7mm_P1.75mm_reverse_mount, F.Cu at (247.7, 97.4)
- added LD36: WS2812B, schizobovine:LED_SK6812MINI_PLCC4_3.1x2.7mm_P1.75mm_reverse_mount, F.Cu at (228.6, 97.4)
- added LD37: WS2812B, schizobovine:LED_SK6812MINI_PLCC4_3.1x2.7mm_P1.75mm_reverse_mount, F.Cu at (209.6, 97.4)
- added LD38: WS2812B, schizobovine:LED_SK6812MINI_PLCC4_3.1x2.7mm_P1.75mm_reverse_mount, F.Cu at (190.5, 97.4)
- added LD39: WS2812B, schizobovine:LED_SK6812MINI_PLCC4_3.1x2.7mm_P1.75mm_reverse_mount, F.Cu at (171.4, 97.4)
- added LD4: WS2812B, schizobovine:LED_SK6812MINI_PLCC4_3.1x2.7mm_P1.75mm_reverse_mount, F.Cu at (228.6, 35.7)
- added LD40: WS2812B, schizobovine:LED_SK6812MINI_PLCC4_3.1x2.7mm_P1.75mm_reverse_mount, F.Cu at (152.4, 97.4)
- added LD41: WS2812B, schizobovine:LED_SK6812MINI_PLCC4_3.1x2.7mm_P1.75mm_reverse_mount, F.Cu at (133.3, 97.4)
- added LD42: WS2812B, schizobovine:LED_SK6812MINI_PLCC4_3.1x2.7mm_P1.75mm_reverse_mount, F.Cu at (114.3, 97.4)
- added LD43: WS2812B, schizobovine:LED_SK6812MINI_PLCC4_3.1x2.7mm_P1.75mm_reverse_mount, F.Cu at (95.2, 97.4)
- added LD44: WS2812B, schizobovine:LED_SK6812MINI_PLCC4_3.1x2.7mm_P1.75mm_reverse_mount, F.Cu at (76.2, 97.4)
- added LD45: WS2812B, schizobovine:LED_SK6812MINI_PLCC4_3.1x2.7mm_P1.75mm_reverse_mount, F.Cu at (57.1, 97.4)
- added LD46: WS2812B, schizobovine:LED_SK6812MINI_PLCC4_3.1x2.7mm_P1.75mm_reverse_mount, F.Cu at (29.2, 97.4)
- added LD47: WS2812B, schizobovine:LED_SK6812MINI_PLCC4_3.1x2.7mm_P1.75mm_reverse_mount, F.Cu at (10.2, 97.4)
- added LD48: WS2812B, schizobovine:LED_SK6812MINI_PLCC4_3.1x2.7mm_P1.75mm_reverse_mount, F.Cu at (10.2, 118.0)
- added LD49: WS2812B, schizobovine:LED_SK6812MINI_PLCC4_3.1x2.7mm_P1.75mm_reverse_mount, F.Cu at (29.2, 118.0)
- added LD5: WS2812B, schizobovine:LED_SK6812MINI_PLCC4_3.1x2.7mm_P1.75mm_reverse_mount, F.Cu at (209.6, 35.7)
- added LD50: WS2812B, schizobovine:LED_SK6812MINI_PLCC4_3.1x2.7mm_P1.75mm_reverse_mount, F.Cu at (61.9, 118.0)
- added LD51: WS2812B, schizobovine:LED_SK6812MINI_PLCC4_3.1x2.7mm_P1.75mm_reverse_mount, F.Cu at (85.7, 118.0)
- added LD52: WS2812B, schizobovine:LED_SK6812MINI_PLCC4_3.1x2.7mm_P1.75mm_reverse_mount, F.Cu at (104.8, 118.0)
- added LD53: WS2812B, schizobovine:LED_SK6812MINI_PLCC4_3.1x2.7mm_P1.75mm_reverse_mount, F.Cu at (123.8, 118.0)
- added LD54: WS2812B, schizobovine:LED_SK6812MINI_PLCC4_3.1x2.7mm_P1.75mm_reverse_mount, F.Cu at (142.9, 118.0)
- added LD55: WS2812B, schizobovine:LED_SK6812MINI_PLCC4_3.1x2.7mm_P1.75mm_reverse_mount, F.Cu at (161.9, 118.0)
- added LD56: WS2812B, schizobovine:LED_SK6812MINI_PLCC4_3.1x2.7mm_P1.75mm_reverse_mount, F.Cu at (181.0, 118.0)
- added LD57: WS2812B, schizobovine:LED_SK6812MINI_PLCC4_3.1x2.7mm_P1.75mm_reverse_mount, F.Cu at (200.0, 118.0)
- added LD58: WS2812B, schizobovine:LED_SK6812MINI_PLCC4_3.1x2.7mm_P1.75mm_reverse_mount, F.Cu at (219.1, 118.0)
- added LD59: WS2812B, schizobovine:LED_SK6812MINI_PLCC4_3.1x2.7mm_P1.75mm_reverse_mount, F.Cu at (238.1, 118.0)
- added LD6: WS2812B, schizobovine:LED_SK6812MINI_PLCC4_3.1x2.7mm_P1.75mm_reverse_mount, F.Cu at (190.5, 35.7)
- added LD60: WS2812B, schizobovine:LED_SK6812MINI_PLCC4_3.1x2.7mm_P1.75mm_reverse_mount, F.Cu at (257.2, 118.0)
- added LD61: WS2812B, schizobovine:LED_SK6812MINI_PLCC4_3.1x2.7mm_P1.75mm_reverse_mount, F.Cu at (276.2, 118.0)
- added LD62: WS2812B, schizobovine:LED_SK6812MINI_PLCC4_3.1x2.7mm_P1.75mm_reverse_mount, F.Cu at (295.3, 118.0)
- added LD63: WS2812B, schizobovine:LED_SK6812MINI_PLCC4_3.1x2.7mm_P1.75mm_reverse_mount, F.Cu at (321.5, 128.3)
- added LD64: WS2812B, schizobovine:LED_SK6812MINI_PLCC4_3.1x2.7mm_P1.75mm_reverse_mount, F.Cu at (351.8, 118.0)
- added LD65: WS2812B, schizobovine:LED_SK6812MINI_PLCC4_3.1x2.7mm_P1.75mm_reverse_mount, F.Cu at (370.8, 118.0)
- added LD66: WS2812B, schizobovine:LED_SK6812MINI_PLCC4_3.1x2.7mm_P1.75mm_reverse_mount, F.Cu at (389.9, 118.0)
- added LD67: WS2812B, schizobovine:LED_SK6812MINI_PLCC4_3.1x2.7mm_P1.75mm_reverse_mount, F.Cu at (417.8, 118.0)
- added LD68: WS2812B, schizobovine:LED_SK6812MINI_PLCC4_3.1x2.7mm_P1.75mm_reverse_mount, F.Cu at (436.9, 118.0)
- added LD69: WS2812B, schizobovine:LED_SK6812MINI_PLCC4_3.1x2.7mm_P1.75mm_reverse_mount, F.Cu at (455.9, 118.0)
- added LD7: WS2812B, schizobovine:LED_SK6812MINI_PLCC4_3.1x2.7mm_P1.75mm_reverse_mount, F.Cu at (171.4, 35.7)
- added LD70: WS2812B, schizobovine:LED_SK6812MINI_PLCC4_3.1x2.7mm_P1.75mm_reverse_mount, F.Cu at (475.0, 128.3)
- added LD71: WS2812B, schizobovine:LED_SK6812MINI_PLCC4_3.1x2.7mm_P1.75mm_reverse_mount, F.Cu at (455.9, 138.5)
- added LD72: WS2812B, schizobovine:LED_SK6812MINI_PLCC4_3.1x2.7mm_P1.75mm_reverse_mount, F.Cu at (436.9, 138.5)
- added LD73: WS2812B, schizobovine:LED_SK6812MINI_PLCC4_3.1x2.7mm_P1.75mm_reverse_mount, F.Cu at (417.8, 138.5)
- added LD74: WS2812B, schizobovine:LED_SK6812MINI_PLCC4_3.1x2.7mm_P1.75mm_reverse_mount, F.Cu at (370.8, 138.5)
- added LD75: WS2812B, schizobovine:LED_SK6812MINI_PLCC4_3.1x2.7mm_P1.75mm_reverse_mount, F.Cu at (300.0, 138.5)
- added LD76: WS2812B, schizobovine:LED_SK6812MINI_PLCC4_3.1x2.7mm_P1.75mm_reverse_mount, F.Cu at (281.0, 138.5)
- added LD77: WS2812B, schizobovine:LED_SK6812MINI_PLCC4_3.1x2.7mm_P1.75mm_reverse_mount, F.Cu at (261.9, 138.5)
- added LD78: WS2812B, schizobovine:LED_SK6812MINI_PLCC4_3.1x2.7mm_P1.75mm_reverse_mount, F.Cu at (242.9, 138.5)
- added LD79: WS2812B, schizobovine:LED_SK6812MINI_PLCC4_3.1x2.7mm_P1.75mm_reverse_mount, F.Cu at (223.8, 138.5)
- added LD8: WS2812B, schizobovine:LED_SK6812MINI_PLCC4_3.1x2.7mm_P1.75mm_reverse_mount, F.Cu at (152.4, 35.7)
- added LD80: WS2812B, schizobovine:LED_SK6812MINI_PLCC4_3.1x2.7mm_P1.75mm_reverse_mount, F.Cu at (204.8, 138.5)
- added LD81: WS2812B, schizobovine:LED_SK6812MINI_PLCC4_3.1x2.7mm_P1.75mm_reverse_mount, F.Cu at (185.7, 138.5)
- added LD82: WS2812B, schizobovine:LED_SK6812MINI_PLCC4_3.1x2.7mm_P1.75mm_reverse_mount, F.Cu at (166.7, 138.5)
- added LD83: WS2812B, schizobovine:LED_SK6812MINI_PLCC4_3.1x2.7mm_P1.75mm_reverse_mount, F.Cu at (147.6, 138.5)
- added LD84: WS2812B, schizobovine:LED_SK6812MINI_PLCC4_3.1x2.7mm_P1.75mm_reverse_mount, F.Cu at (128.6, 138.5)
- added LD85: WS2812B, schizobovine:LED_SK6812MINI_PLCC4_3.1x2.7mm_P1.75mm_reverse_mount, F.Cu at (109.5, 138.5)
- added LD86: WS2812B, schizobovine:LED_SK6812MINI_PLCC4_3.1x2.7mm_P1.75mm_reverse_mount, F.Cu at (90.5, 138.5)
- added LD87: WS2812B, schizobovine:LED_SK6812MINI_PLCC4_3.1x2.7mm_P1.75mm_reverse_mount, F.Cu at (70.5, 128.8)
- added LD88: WS2812B, schizobovine:LED_SK6812MINI_PLCC4_3.1x2.7mm_P1.75mm_reverse_mount, F.Cu at (52.6, 139.9)
- added LD89: WS2812B, schizobovine:LED_SK6812MINI_PLCC4_3.1x2.7mm_P1.75mm_reverse_mount, F.Cu at (29.2, 138.5)
- added LD9: WS2812B, schizobovine:LED_SK6812MINI_PLCC4_3.1x2.7mm_P1.75mm_reverse_mount, F.Cu at (133.3, 35.7)
- added LD90: WS2812B, schizobovine:LED_SK6812MINI_PLCC4_3.1x2.7mm_P1.75mm_reverse_mount, F.Cu at (10.2, 138.5)
- added LD91: WS2812B, schizobovine:LED_SK6812MINI_PLCC4_3.1x2.7mm_P1.75mm_reverse_mount, F.Cu at (10.2, 159.1)
- added LD92: WS2812B, schizobovine:LED_SK6812MINI_PLCC4_3.1x2.7mm_P1.75mm_reverse_mount, F.Cu at (29.2, 159.1)
- added LD93: WS2812B, schizobovine:LED_SK6812MINI_PLCC4_3.1x2.7mm_P1.75mm_reverse_mount, F.Cu at (69.1, 159.1)
- added LD94: WS2812B, schizobovine:LED_SK6812MINI_PLCC4_3.1x2.7mm_P1.75mm_reverse_mount, F.Cu at (100.0, 159.1)
- added LD95: WS2812B, schizobovine:LED_SK6812MINI_PLCC4_3.1x2.7mm_P1.75mm_reverse_mount, F.Cu at (119.1, 159.1)
- added LD96: WS2812B, schizobovine:LED_SK6812MINI_PLCC4_3.1x2.7mm_P1.75mm_reverse_mount, F.Cu at (138.1, 159.1)
- added LD97: WS2812B, schizobovine:LED_SK6812MINI_PLCC4_3.1x2.7mm_P1.75mm_reverse_mount, F.Cu at (157.2, 159.1)
- added LD98: WS2812B, schizobovine:LED_SK6812MINI_PLCC4_3.1x2.7mm_P1.75mm_reverse_mount, F.Cu at (176.2, 159.1)
- added LD99: WS2812B, schizobovine:LED_SK6812MINI_PLCC4_3.1x2.7mm_P1.75mm_reverse_mount, F.Cu at (195.3, 159.1)
- added U2: SN74LVC1G125DBV, Package_TO_SOT_SMD:SOT-23-5, B.Cu at (302.2, 36.0)
- MX008: footprint MX_Only:MXOnly-1U-Hotswap-LED -> MX_Only:MXOnly-1U-Hotswap
- MX041: value MX-LED -> MX-NoLED; footprint MX_Only:MXOnly-1.75U -> MX_Only:MXOnly-1.75U-Hotswap
- MX041.125: value MX-LED -> MX-NoLED; footprint MX_Only:MXOnly-1.25U-Hotswap-LED -> MX_Only:MXOnly-1.25U-Hotswap
- N1: renamed from Solenoid; value solenoid -> Solenoid; footprint redherring:solenoid -> schizobovine:solenoid
- moved D46 5.17 mm to (421.1, 184.2)
- turned MX041 to 180 degrees
- turned MX087.200 to 0 degrees
- turned MX117.100 to 0 degrees
Connections:
- D10 pad 2: Net-(MX121-ROW) -> unconnected-(D10-A-Pad2)
- D47 pad 2: Net-(MX077-ROW) -> unconnected-(D47-A-Pad2)
- D53 pad 1: Net-(MX136-ROW) -> unconnected-(D53-A-Pad1)
- D53 pad 2: Net-(MX137-ROW) -> unconnected-(D53-A-Pad2)
- D63 pad 2: Net-(MX099-ROW) -> unconnected-(D63-A-Pad2)
- U1 pad 6: unconnected-(U1-PA9-Pad6) -> RGB_3v3
- U1 pad 7: BL_BUZ -> unconnected-(U1-PA10-Pad7)
Routing:
- net SCK_CAPS: track 490.5 -> 27.5 mm, vias 3 -> 0
- net BL_BUZ: track 101.3 -> 0.00 mm, vias 2 -> 0
- net Net-(MX077-ROW): track 88.8 -> 0.00 mm, vias 2 -> 0
- net Net-(MX063-ROW): track 76.3 -> 0.00 mm
- net COL7: track 716.0 -> 786.2 mm, vias 8 -> 11
- net MOSI_NUM: track 103.8 -> 36.5 mm, vias 4 -> 0
- net unconnected-(D63-A-Pad2): track 0.00 -> 41.7 mm
- net Net-(MX137-ROW): track 41.0 -> 0.00 mm
- net Net-(MX099-ROW): track 38.5 -> 0.00 mm
- net unconnected-(D10-A-Pad2): track 0.00 -> 36.6 mm
- net Net-(MX121-ROW): track 36.6 -> 0.00 mm
- net COL2: track 729.3 -> 695.2 mm
- net COL6: track 650.5 -> 618.1 mm
- net Net-(MX062-ROW): track 23.7 -> 0.00 mm
- net (no net): track 0.00 -> 23.7 mm
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Other:
- board text added: "(Rev 2.moo)"
- board text added: "Designed by dcpedit minor edits by schizobovine github.com/seancaulfield/mission-control"
- board text removed: "(Rev 2)"
- board text removed: "Designed by dcpedit github.com/dcpedit/mission-control"
