File: pcb/pcb.kicad_pcb (KiCad board)
At the start: 2 copper layers, 489.6 x 170.7 mm, 390 parts, among them J1 Conn_01x08_Socket, J2 Conn_01x02_Female, U1 YAAJ_WeAct_BlackPill_Part_Lik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, U2 SN74LVC1G125DBV

Commit message: RGB added
Parts:
- removed D53: BAV70, Keebio-Parts:SOT-23_Handsoldering
- removed H54, H56: MountingHole, MountingHole:MountingHole_3mm
- removed MX127: MX-NoLED, MX_Only:MXOnly-2.75U-Hotswap
- added D18: BAV70, Keebio-Parts:SOT-23_Handsoldering, B.Cu at (135.1, 175.7)
- added FID2: Fiducial, schizobovine:oshw, B.Cu at (229.0, 177.2)
- added FID3: Fiducial, schizobovine:qmk_logo, F.Cu at (217.7, 175.9)
- added FID4: Fiducial, schizobovine:qmk_logo, B.Cu at (162.5, 175.9)
- added FID5: Fiducial, schizobovine:COW, B.Cu at (207.9, 178.2)
- added G***: LOGO, mc:control, B.Cu at (163.3, 70.1)
- added G***: LOGO, mc:mission, B.Cu at (238.3, 70.1)
- added H100: MountingHole, schizobovine:MountingHole_3.1mm_M2.5_solderable, F.Cu at (410.7, 181.3)
- added H101: MountingHole, schizobovine:MountingHole_3.1mm_M2.5_solderable, F.Cu at (266.7, 168.1)
- added H108: MountingHole, schizobovine:MountingHole_3.1mm_M2.5_solderable, F.Cu at (361.3, 147.6)
- added H110: MountingHole, schizobovine:MountingHole_3.1mm_M2.5_solderable, F.Cu at (85.7, 24.1)
- added H111: MountingHole, schizobovine:MountingHole_3.1mm_M2.5_solderable, F.Cu at (161.9, 24.1)
- added H112: MountingHole, schizobovine:MountingHole_3.1mm_M2.5_solderable, F.Cu at (200.0, 44.5)
- added H113: MountingHole, schizobovine:MountingHole_3.1mm_M2.5_solderable, F.Cu at (85.7, 58.2)
- added H114: MountingHole, schizobovine:MountingHole_3.1mm_M2.5_solderable, F.Cu at (181.0, 58.2)
- added H115: MountingHole, schizobovine:MountingHole_3.1mm_M2.5_solderable, F.Cu at (276.2, 58.2)
- added H116: MountingHole, schizobovine:MountingHole_3.1mm_M2.5_solderable, F.Cu at (345.0, 102.8)
- added H117: MountingHole, schizobovine:MountingHole_3.1mm_M2.5_solderable, F.Cu at (19.7, 181.5)
- added H118: MountingHole, schizobovine:MountingHole_3.1mm_M2.5_solderable, F.Cu at (19.7, 127.1)
- added H119: MountingHole, schizobovine:MountingHole_3.1mm_M2.5_solderable, F.Cu at (19.7, 168.1)
- added H120: MountingHole, schizobovine:MountingHole_3.1mm_M2.5_solderable, F.Cu at (114.3, 181.8)
- added H121: MountingHole, schizobovine:MountingHole_3.1mm_M2.5_solderable, F.Cu at (266.7, 181.5)
- added H122: MountingHole, schizobovine:MountingHole_3.1mm_M2.5_solderable, F.Cu at (164.2, 181.5)
- added H123: MountingHole, schizobovine:MountingHole_3.1mm_M2.5_solderable, F.Cu at (217.4, 181.5)
- added H124: MountingHole, schizobovine:MountingHole_3.1mm_M2.5_solderable, F.Cu at (329.5, 180.5)
- added H125: MountingHole, schizobovine:MountingHole_3.1mm_M2.5_solderable, F.Cu at (72.7, 181.5)
- added H70: MountingHole, schizobovine:MountingHole_3.1mm_M2.5_solderable, F.Cu at (114.3, 168.1)
- added H71: MountingHole, schizobovine:MountingHole_3.1mm_M2.5_solderable, F.Cu at (50.0, 106.2)
- added H74: MountingHole, schizobovine:MountingHole_3.1mm_M2.5_solderable, F.Cu at (380.3, 161.0)
- added H75: MountingHole, schizobovine:MountingHole_3.1mm_M2.5_solderable, F.Cu at (380.4, 85.6)
- added H76: MountingHole, schizobovine:MountingHole_3.1mm_M2.5_solderable, F.Cu at (361.4, 161.0)
- added H77: MountingHole, schizobovine:MountingHole_3.1mm_M2.5_solderable, F.Cu at (465.5, 85.8)
- added H78: MountingHole, schizobovine:MountingHole_3.1mm_M2.5_solderable, F.Cu at (427.4, 106.4)
- added H79: MountingHole, schizobovine:MountingHole_3.1mm_M2.5_solderable, F.Cu at (446.3, 144.0)
- added H81: MountingHole, schizobovine:MountingHole_3.1mm_M2.5_solderable, F.Cu at (410.7, 164.7)
- added H82: MountingHole, schizobovine:MountingHole_3.1mm_M2.5_solderable, F.Cu at (50.0, 147.6)
- added H83: MountingHole, schizobovine:MountingHole_3.1mm_M2.5_solderable, F.Cu at (396.5, 102.8)
- added H84: MountingHole, schizobovine:MountingHole_3.1mm_M2.5_solderable, F.Cu at (427.4, 85.8)
- added H85: MountingHole, schizobovine:MountingHole_3.1mm_M2.5_solderable, F.Cu at (483.0, 144.0)
- added H86: MountingHole, schizobovine:MountingHole_3.1mm_M2.5_solderable, F.Cu at (446.3, 181.3)
- added H87: MountingHole, schizobovine:MountingHole_3.1mm_M2.5_solderable, F.Cu at (483.0, 106.4)
- added H88: MountingHole, schizobovine:MountingHole_3.1mm_M2.5_solderable, F.Cu at (483.0, 181.3)
- added H89: MountingHole, schizobovine:MountingHole_3.1mm_M2.5_solderable, F.Cu at (446.4, 164.7)
- added H90: MountingHole, schizobovine:MountingHole_3.1mm_M2.5_solderable, F.Cu at (361.3, 120.6)
- added H91: MountingHole, schizobovine:MountingHole_3.1mm_M2.5_solderable, F.Cu at (329.5, 106.3)
- added H95: MountingHole, schizobovine:MountingHole_3.1mm_M2.5_solderable, F.Cu at (329.5, 127.2)
- added H96: MountingHole, schizobovine:MountingHole_3.1mm_M2.5_solderable, F.Cu at (380.2, 120.6)
- added H97: MountingHole, schizobovine:MountingHole_3.1mm_M2.5_solderable, F.Cu at (329.5, 147.6)
- added H98: MountingHole, schizobovine:MountingHole_3.1mm_M2.5_solderable, F.Cu at (410.7, 144.0)
- added LD123: WS2812B, schizobovine:LED_SK6812MINI_PLCC4_3.1x2.7mm_P1.75mm_reverse_mount, F.Cu at (304.8, 97.4)
- added LD124: WS2812B, schizobovine:LED_SK6812MINI_PLCC4_3.1x2.7mm_P1.75mm_reverse_mount, F.Cu at (104.8, 179.7)
- added LD125: WS2812B, schizobovine:LED_SK6812MINI_PLCC4_3.1x2.7mm_P1.75mm_reverse_mount, F.Cu at (257.2, 179.7)
- added MX077: MX-NoLED, MX_Only:MXOnly-1U-Hotswap, F.Cu at (304.8, 92.5)
- added MX10: MX-NoLED, MX_Only:MXOnly-1U-Hotswap, F.Cu at (123.8, 174.8)
- added MX11: MX-NoLED, MX_Only:MXOnly-1U-Hotswap, F.Cu at (257.2, 174.8)
- H10, H17, H18, H19, H2, H20, H21, H22, H24, H25, H26, H27, H28, H29, H3, H32, H34, H36, H37, H38, H4, H42, H44, H45, H46, H47, H48, H5, H50, H53, H55, H57, H8, H9: footprint MountingHole:MountingHole_3mm -> schizobovine:MountingHole_3.1mm_M2.5_solderable
- MX047: renamed from MX047.200; footprint MX_Only:MXOnly-ISO-Hotswap -> MX_Only:MXOnly-2.25U-Hotswap-ReversedStabilizers
- MX087: renamed from MX087.200; footprint MX_Only:MXOnly-2U-Hotswap-ReversedStabilizers -> MX_Only:MXOnly-1U-Hotswap
- MX117: renamed from MX117.100; footprint MX_Only:MXOnly-1U-Hotswap -> MX_Only:MXOnly-1.5U-Hotswap
- MX131, MX133: footprint MX_Only:MXOnly-1.5U-Hotswap -> MX_Only:MXOnly-1U-Hotswap
- MX132: footprint MX_Only:MXOnly-7U-Hotswap -> MX_Only:MXOnly-6U-Centered-Hotswap
- moved FID1 226.8 mm to (396.8, 134.2)
- moved MX117 28.0 mm to (319.1, 113.1)
- moved LD119 14.3 mm to (123.8, 179.7)
- moved MX047 14.0 mm to (311.9, 133.6)
- moved LD75 11.9 mm to (311.9, 138.5)
- moved LD63 10.6 mm to (319.1, 118.0)
- moved LD104 9.80 mm to (290.5, 159.1)
- moved LD105 9.53 mm to (316.7, 159.1), turned to 180 degrees
- moved LD32 9.53 mm to (323.9, 97.4)
- moved MX087 9.53 mm to (323.9, 92.5)
- moved LD117 4.76 mm to (276.2, 179.7)
- moved MX133 4.76 mm to (276.2, 174.8)
- moved MX131 4.76 mm to (104.8, 174.8)
- moved D25 4.00 mm to (219.1, 175.0)
- moved LD88 2.47 mm to (54.5, 138.4), turned to -90 degrees
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Connections:
- D47 pad 2: unconnected-(D47-A-Pad2) -> Net-(MX077-ROW)
- D52 pad 2: Net-(MX127-ROW) -> Net-(MX127.175-ROW)
- LD118 pad 4: Net-(LD117-DOUT) -> Net-(LD118-DIN)
- LD120 pad 4: Net-(LD119-DOUT) -> Net-(LD120-DIN)
- LD32 pad 2: Net-(LD32-DOUT) -> Net-(LD123-DIN)
- LD33 pad 4: Net-(LD32-DOUT) -> Net-(LD123-DOUT)
- MX127.175 pad 2: COL7 -> Net-(MX127.175-ROW)
Routing:
- net +5V: track 69.7 -> 4128.0 mm, vias 2 -> 280
- net Net-(LD24-DOUT): track 0.00 -> 223.2 mm, vias 0 -> 6
- net RGB_3v3: track 0.00 -> 164.9 mm, vias 0 -> 1
- net Net-(MX11-ROW): track 0.00 -> 134.2 mm
- net Net-(MX077-ROW): track 0.00 -> 83.4 mm, vias 0 -> 2
- net Net-(LD118-DIN): track 0.00 -> 69.9 mm
- net Net-(LD118-DOUT): track 0.00 -> 63.8 mm
- net Net-(LD74-DOUT): track 0.00 -> 54.3 mm, vias 0 -> 2
- net Net-(MX127.175-ROW): track 0.00 -> 53.3 mm
- net ROW13: track 597.1 -> 544.0 mm
- net Net-(LD114-DOUT): track 0.00 -> 51.9 mm
- net Net-(LD115-DOUT): track 0.00 -> 49.7 mm, vias 0 -> 4
- net Net-(LD73-DOUT): track 0.00 -> 44.4 mm
- net unconnected-(D63-A-Pad2): track 41.7 -> 0.00 mm
- net Net-(LD65-DOUT): track 0.00 -> 40.9 mm, vias 0 -> 2
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Other:
- board size 489.6 x 170.7 mm -> 489.6 x 171.7 mm
- board text added: "(Rev 3.cowabunga)"
- board text added: "Battlecruiser operational"
- board text added: "Designed by dcpedit bling bling added by schizobovine github.com/dcpedit/mission-control github.com/seancaulfield/mission-control"
- board text added: "M122ION CONTROL RAVE EDITION"
- board text added: "RAVE EDITION"
- board text removed: "(Rev 2.moo)"
- board text removed: "Designed by dcpedit minor edits by schizobovine github.com/seancaulfield/mission-control"
- board text removed: "M122ION CONTROL"
