File: pcb/pcb.kicad_pcb (KiCad board)
At the start: 2 copper layers, 489.6 x 171.7 mm, 441 parts, among them J1 Conn_01x08_Socket, J2 Conn_01x02_Female, U1 YAAJ_WeAct_BlackPill_Part_Lik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, U2 SN74LVC1G125DBV

Commit message: finished RGB
Parts:
- added J3: Aux 5V, TerminalBlock:TerminalBlock_bornier-2_P5.08mm, B.Cu at (362.5, 26.5)
- added J4: Aux 5V, Connector_Wire:SolderWire-2sqmm_1x02_P7.8mm_D2mm_OD3.9mm, F.Cu at (362.5, 33.0)
Routing:
- net +5V: track 4128.0 -> 4138.1 mm
- net ROW7: track 476.0 -> 470.4 mm
- net ROW8: track 470.3 -> 466.3 mm
- net COL6: track 624.8 -> 621.4 mm
- net COL7: track 746.4 -> 742.9 mm
- net COL4: track 736.1 -> 733.0 mm
- net COL3: track 708.1 -> 709.0 mm
- net COL2: track 699.8 -> 700.6 mm
- net ROW9: track 571.2 -> 572.0 mm
- net ROW2: track 547.4 -> 548.2 mm
- net COL1: track 653.9 -> 654.7 mm
- net COL0: track 690.9 -> 691.6 mm
- net ROW0: track 466.7 -> 467.3 mm
- net RGB_3v3: track 164.9 -> 164.7 mm, vias 1 -> 2
Other:
- board text added: "Ext 5V"
